File: pcb/TwoWheelRobotPCB/Supply.kicad_sch (KiCad schematic)
At the start: 0 parts

Commit message: pcb
Parts:
- added C10: 0.1uF, Capacitor_THT:C_Disc_D4.3mm_W1.9mm_P5.00mm, symbol cyclophone:C
- added C11: 680uF, Capacitor_SMD:CP_Elec_8x6.9, symbol Device:C_Polarized
- added C12: 220uF, Capacitor_SMD:CP_Elec_8x6.9, symbol Device:C_Polarized
- added C9: 100uF, Capacitor_THT:CP_Radial_D6.3mm_P2.50mm, symbol Device:C_Polarized
- added D9: 1N5825, Diode_SMD:D_2010_5025Metric_Pad1.52x2.65mm_HandSolder, symbol Diode:1N5822
- added J3: POWER, TerminalBlock_RND:TerminalBlock_RND_205-00001_1x02_P5.00mm_Horizontal, symbol Connector:Screw_Terminal_01x02
- added J4: XT60-M, footprint:AMASS_XT60-M, symbol XT60-M:XT60-M
- added L1: 33uH, Inductor_SMD:L_Bourns_SRP1245A, symbol Device:L
- added SW1: SW_DPDT_x2, Button_Switch_THT:SW_PUSH_E-Switch_FS5700DP_DPDT, symbol Switch:SW_DPDT_x2
- added U9: LM2596S-5, Package_TO_SOT_SMD:TO-263-5_TabPin3, symbol Regulator_Switching:LM2596S-5
Connections:
- net +5V: now also C12.1, L1.1, U9.4 (FB)
- net GND: now also C10.1, C11.2, C12.2, C9.2, D9.2 (A), J3.2 (Pin_2), J4.N (NEG), U9.3 (GND), U9.5 (~{ON}/OFF)
- net VS: now also C10.2, C11.1, C9.1, SW1.3 (C), U9.1 (VIN)
- new net: J3.1 (Pin_1), J4.P (POS), SW1.2 (B)
- new net: D9.1 (K), L1.2, U9.2 (OUT)
- no-connect marks 0 -> 1
