File: pcb/TwoWheelRobotPCB/MotorDriver.kicad_sch (KiCad schematic)
At the start: 23 parts, among them J1 L298n_sense_connector, J2 ACS712_connector, J3 Motor1, J4 Motor2, U2 L298HN, U3 PCF8574, U4 TXB0108DQSR

Commit message: update pcb
Parts:
- removed J1: L298n_sense_connector, Connector_PinHeader_2.54mm:PinHeader_2x02_P2.54mm_Vertical, symbol Connector_Generic:Conn_02x02_Counter_Clockwise
- removed J2: ACS712_connector, Connector_PinHeader_2.54mm:PinHeader_2x02_P2.54mm_Vertical, symbol Connector_Generic:Conn_02x02_Counter_Clockwise
Connections:
- net dir1_M1: now also U3.7 (P3); no longer U3.4 (P0)
- net dir1_M2: now also U3.6 (P2); no longer U3.5 (P1)
- net dir2_M1: now also U3.5 (P1); no longer U3.6 (P2)
- net dir2_M2: now also U3.4 (P0); no longer U3.7 (P3)

Commit message: pcb
Parts:
- removed U4: TXB0108DQSR, TXB0108_TSOP20_fotprint:SOP65P640X120-20N, symbol Logic_LevelTranslator:TXB0108DQSR
- added U4: TXB0108PWR, TXB0108_TSOP20_fotprint:SOP65P640X120-20N, symbol TXB0108PWR:TXB0108PWR
- renumbered J3 to J1, J4 to J2
Connections:
- net +3V3: now also U4.10 (OE), U4.2 (VCCA)
- net +5V: now also U4.19 (VCCB)
- net DIR1_M1: now also U4.18 (B2)
- net DIR1_M2: now also U4.17 (B3)
- net DIR2_M1: now also U4.16 (B4)
- net DIR2_M2: now also U4.15 (B5)
- net GND: now also U4.11 (GND)
- net PWM1: now also U4.20 (B1)
- net PWM2: now also U4.14 (B6)
- net dir1_M1 renamed dir1_M1_3v3
- net dir1_M1_3v3: now also U4.3 (A2)
- net dir1_M2 renamed dir1_M2_3v3
- net dir1_M2_3v3: now also U4.4 (A3)
- net dir2_M1 renamed dir2_M1_3v3
- net dir2_M1_3v3: now also U4.5 (A4)
- net dir2_M2 renamed dir2_M2_3v3
- net dir2_M2_3v3: now also U4.6 (A5)
- new net pwm1_3v3: U4.1 (A1)
- new net pwm2_3v3: U4.7 (A6)

Commit message: pcb finish
Parts:
- renumbered D2 to D1, D1 to D2, D4 to D3, D3 to D4, D6 to D5, D5 to D6, D8 to D7, D7 to D8
Changed lines of the file:
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@@
   (symbol (lib_id "pspice:DIODE") (at 96.52 101.6 90) (unit 1)
     (in_bom yes) (on_board yes)
-    (property "Reference" "D6" (id 0) (at 96.52 97.79 90)
+    (property "Reference" "D5" (id 0) (at 96.52 97.79 90)
       (effects (font (size 1.27 1.27)) (justify right))
     )
@@
   (symbol (lib_id "pspice:DIODE") (at 104.14 101.6 90) (unit 1)
     (in_bom yes) (on_board yes)
-    (property "Reference" "D8" (id 0) (at 104.14 97.79 90)
+    (property "Reference" "D7" (id 0) (at 104.14 97.79 90)
       (effects (font (size 1.27 1.27)) (justify right))
     )
@@
   (symbol (lib_id "pspice:DIODE") (at 88.9 101.6 90) (unit 1)
     (in_bom yes) (on_board yes)
-    (property "Reference" "D4" (id 0) (at 88.9 97.79 90)
+    (property "Reference" "D3" (id 0) (at 88.9 97.79 90)
       (effects (font (size 1.27 1.27)) (justify right))
     )
@@
   (symbol (lib_id "pspice:DIODE") (at 104.14 78.74 90) (unit 1)
     (in_bom yes) (on_board yes)
-    (property "Reference" "D7" (id 0) (at 104.14 74.93 90)
+    (property "Reference" "D8" (id 0) (at 104.14 74.93 90)
       (effects (font (size 1.27 1.27)) (justify right))
     )
@@
   (symbol (lib_id "pspice:DIODE") (at 88.9 78.74 90) (unit 1)
     (in_bom yes) (on_board yes)
-    (property "Reference" "D3" (id 0) (at 88.9 74.93 90)
+    (property "Reference" "D4" (id 0) (at 88.9 74.93 90)
       (effects (font (size 1.27 1.27)) (justify right))
     )
@@
   (symbol (lib_id "pspice:DIODE") (at 96.52 78.74 90) (unit 1)
     (in_bom yes) (on_board yes)
-    (property "Reference" "D5" (id 0) (at 96.52 74.93 90)
+    (property "Reference" "D6" (id 0) (at 96.52 74.93 90)
       (effects (font (size 1.27 1.27)) (justify right))
     )
@@
   (symbol (lib_id "pspice:DIODE") (at 81.28 101.6 90) (unit 1)
     (in_bom yes) (on_board yes)
-    (property "Reference" "D2" (id 0) (at 81.28 97.79 90)
+    (property "Reference" "D1" (id 0) (at 81.28 97.79 90)
       (effects (font (size 1.27 1.27)) (justify right))
     )
@@
   (symbol (lib_id "pspice:DIODE") (at 81.28 78.74 90) (unit 1)
     (in_bom yes) (on_board yes)
-    (property "Reference" "D1" (id 0) (at 81.28 74.93 90)
-      (effects (font (size 1.27 1.27)) (justify right))
-    )
+    (property "Reference" "D2" (id 0) (at 81.28 74.93 90)
+      (effects (font (size 1.27 1.27)) (justify right))
+    )
