File: pcb/TwoWheelRobotPCB/TwoWheelRobotPCB.kicad_pcb (KiCad board)
At the start: 2 copper layers, 8 parts, among them J1 Motor1, J2 Motor2, J3 L298n_sense_connector, J4 ACS712_connector, U2 L298HN, U3 ACS712_M1, U4 TXB0104D, U5 ACS712_M2

Commit message: pcb update
Parts:
- added C1: 100uF, Capacitor_THT:CP_Radial_D6.3mm_P2.50mm, F.Cu at (132.0, 85.5)
- added C2: 0.1uF, Capacitor_THT:C_Disc_D4.3mm_W1.9mm_P5.00mm, F.Cu at (131.5, 82.0)
- added C3: 100uF, Capacitor_THT:CP_Radial_D6.3mm_P2.50mm, F.Cu at (113.0, 80.6)
- added C4: 0.1uF, Capacitor_THT:C_Disc_D4.3mm_W1.9mm_P5.00mm, F.Cu at (118.0, 84.5)
- added C5: 0.1uF, Capacitor_SMD:C_0805_2012Metric, F.Cu at (89.0, 83.0)
- added C6: 0.1uF, Capacitor_SMD:C_0805_2012Metric, F.Cu at (175.5, 89.0)
- added C7: 1nF, Capacitor_SMD:C_0805_2012Metric, F.Cu at (89.0, 87.2)
- added C8: 1nF, Capacitor_SMD:C_0805_2012Metric, F.Cu at (168.0, 95.5)
- added D1: DIODE, Diode_THT:D_A-405_P10.16mm_Horizontal, F.Cu at (116.1, 67.2)
- added D2: DIODE, Diode_THT:D_A-405_P10.16mm_Horizontal, F.Cu at (105.9, 64.0)
- added D3: DIODE, Diode_THT:D_A-405_P10.16mm_Horizontal, F.Cu at (116.1, 75.8)
- added D4: DIODE, Diode_THT:D_A-405_P10.16mm_Horizontal, F.Cu at (105.9, 72.5)
- added D5: DIODE, Diode_THT:D_A-405_P10.16mm_Horizontal, F.Cu at (143.8, 72.5)
- added D6: DIODE, Diode_THT:D_A-405_P10.16mm_Horizontal, F.Cu at (154.0, 75.8)
- added D7: DIODE, Diode_THT:D_A-405_P10.16mm_Horizontal, F.Cu at (143.8, 64.0)
- added D8: DIODE, Diode_THT:D_A-405_P10.16mm_Horizontal, F.Cu at (154.0, 67.2)
- added R1: Rsa, Resistor_SMD:R_0805_2012Metric, F.Cu at (121.0, 82.5)
- added R2: Rsb, Resistor_SMD:R_0805_2012Metric, F.Cu at (139.0, 82.5)
- added R3: 10k, Resistor_SMD:R_0805_2012Metric, F.Cu at (109.0, 117.0)
- added R4: 18k, Resistor_SMD:R_0805_2012Metric, F.Cu at (112.0, 114.0)
- added R5: 2k2, Resistor_SMD:R_0805_2012Metric, F.Cu at (145.0, 118.2)
- added R6: 2k2, Resistor_SMD:R_0805_2012Metric, F.Cu at (147.0, 118.2)
- added REF**: MountingHole_2.2mm_M2_DIN965_Pad, MountingHole:MountingHole_2.2mm_M2_DIN965_Pad, F.Cu at (177.5, 157.5)
- added REF**: MountingHole_2.2mm_M2_DIN965_Pad, MountingHole:MountingHole_2.2mm_M2_DIN965_Pad, F.Cu at (82.5, 157.5)
- added REF**: MountingHole_2.2mm_M2_DIN965_Pad, MountingHole:MountingHole_2.2mm_M2_DIN965_Pad, F.Cu at (82.5, 62.5)
- added REF**: Heatsink_Fischer_SK104-STC-STIC_35x13mm_2xDrill2.5mm, Heatsink:Heatsink_Fischer_SK104-STC-STIC_35x13mm_2xDrill2.5mm, F.Cu at (130.0, 67.2)
- added REF**: MountingHole_2.2mm_M2_DIN965_Pad, MountingHole:MountingHole_2.2mm_M2_DIN965_Pad, F.Cu at (177.5, 62.5)
- added U1: NodeMCU1.0(ESP-12E), NodemcuESP8266_footprint:MODULE_ZC563900, F.Cu at (130.0, 135.5)
- added U6: MCP3004, MCP3004_footprint:SOIC127P600X175-14N, F.Cu at (130.0, 110.0)
- added U7: ACS712_M1, Package_SO:SOIC-8_3.9x4.9mm_P1.27mm, F.Cu at (98.5, 73.8)
- added U8: ACS712_M2, Package_SO:SOIC-8_3.9x4.9mm_P1.27mm, F.Cu at (159.8, 73.5)
- J1: value Motor1 -> L298n_sense_connector; footprint Connector_PinHeader_2.54mm:PinHeader_1x06_P2.54mm_Vertical -> Connector_PinHeader_2.54mm:PinHeader_2x02_P2.54mm_Vertical
- J2: value Motor2 -> ACS712_connector; footprint Connector_PinHeader_2.54mm:PinHeader_1x06_P2.54mm_Vertical -> Connector_PinHeader_2.54mm:PinHeader_2x02_P2.54mm_Vertical
- J3: value L298n_sense_connector -> Motor1; footprint Connector_PinHeader_2.54mm:PinHeader_2x02_P2.54mm_Vertical -> Connector_PinHeader_2.54mm:PinHeader_1x06_P2.54mm_Vertical
- J4: value ACS712_connector -> Motor2; footprint Connector_PinHeader_2.54mm:PinHeader_2x02_P2.54mm_Vertical -> Connector_PinHeader_2.54mm:PinHeader_1x06_P2.54mm_Vertical
- U3: value ACS712_M1 -> PCF8574; footprint Package_SO:SOIC-8_3.9x4.9mm_P1.27mm -> PCF8574:SO16W
- U4: value TXB0104D -> TXB0108DQSR; footprint Package_SO:SOIC-14_3.9x8.7mm_P1.27mm -> TXB0108_TSOP20_fotprint:SOP65P640X120-20N
- U5: value ACS712_M2 -> TXB0104D; footprint Package_SO:SOIC-8_3.9x4.9mm_P1.27mm -> TXB0104_TSOP14_footprint:SOP65P640X120-14N
- moved J3 45.1 mm to (90.2, 67.2), turned to 90 degrees
- moved U5 45.0 mm to (130.0, 125.0), turned to 90 degrees
- moved J4 37.3 mm to (170.8, 67.2), turned to -90 degrees
- moved J2 36.1 mm to (131.5, 101.0)
- moved U3 34.4 mm to (113.0, 91.8), turned to 90 degrees
- moved J1 24.8 mm to (105.0, 81.8)
- moved U4 22.2 mm to (124.8, 89.2), turned to 90 degrees
- moved U2 19.8 mm to (121.1, 79.5)
Connections:
- J1 pad 1: unconnected-(J1-Pad1) -> ADC1
- J1 pad 2: unconnected-(J1-Pad2) -> ADC2
- J1 pad 3: unconnected-(J1-Pad3) -> Sense_B
- J1 pad 4: unconnected-(J1-Pad4) -> Sense_A
- J2 pad 1: unconnected-(J2-Pad1) -> ADC1
- J2 pad 2: unconnected-(J2-Pad2) -> ADC2
- J2 pad 3: unconnected-(J2-Pad3) -> VIOUT_M2
- J2 pad 4: unconnected-(J2-Pad4) -> VIOUT_M1
- J3 pad 1: ADC1 -> M1-
- J3 pad 2: ADC2 -> GND
- J3 pad 3: Sense_B -> M1_C1
- J3 pad 4: Sense_A -> M1_C2
- J4 pad 1: ADC1 -> M2-
- J4 pad 2: ADC2 -> GND
- J4 pad 3: VIOUT_M2 -> M2_C1
- J4 pad 4: VIOUT_M1 -> M2_C2
- U2 pad 13: OUT3 -> OUT2
- U2 pad 14: OUT4 -> M2-
- U2 pad 3: OUT2 -> M1-
- U2 pad 9: +3V3 -> +5V
- U3 pad 1: Net-(U3-Pad1) -> GND
- U3 pad 2: Net-(U3-Pad1) -> GND
- U3 pad 3: Net-(U3-Pad3) -> GND
- U3 pad 4: Net-(U3-Pad3) -> dir1_M1
- U3 pad 5: GND -> dir1_M2
- U3 pad 6: Net-(U3-Pad6) -> dir2_M1
- U3 pad 7: VIOUT_M1 -> dir2_M2
- U3 pad 8: +5V -> GND
- U4 pad 1: +3V3 -> pwm1
- U4 pad 10: CS -> unconnected-(U4-Pad10)
- U4 pad 11: Din -> unconnected-(U4-Pad11)
- U4 pad 12: Dout -> unconnected-(U4-Pad12)
- U4 pad 13: CLK -> PWM2
- U4 pad 14: +5V -> DIR2_M2
- U4 pad 2: SCLK -> dir1_M1
- U4 pad 3: MISO -> dir1_M2
- U4 pad 4: MOSI -> dir2_M1
- U4 pad 5: CS_ -> +3V3
- U4 pad 6: unconnected-(U4-Pad6) -> +3V3
- U4 pad 7: GND -> dir2_M2
- U4 pad 8: +3V3 -> pwm2
- U5 pad 1: Net-(U5-Pad1) -> +3V3
- U5 pad 2: Net-(U5-Pad1) -> MOSI
- U5 pad 3: Net-(U5-Pad3) -> CS_
- U5 pad 4: Net-(U5-Pad3) -> MISO
- U5 pad 5: GND -> SCLK
- U5 pad 6: Net-(C8-Pad1) -> unconnected-(U5-Pad6)
- U5 pad 7: VIOUT_M2 -> GND
- U5 pad 8: +5V -> +3V3
Routing:
- net VS: track 0.00 -> 45.7 mm
- net Sense_B: track 0.00 -> 35.6 mm, vias 0 -> 1
- net SCLK: track 0.00 -> 17.7 mm
- net Din: track 0.00 -> 17.2 mm
- net Sense_A: track 0.00 -> 16.8 mm
- net DIR1_M2: track 0.00 -> 16.7 mm
- net DIR2_M2: track 0.00 -> 16.7 mm
- net PWM2: track 0.00 -> 16.4 mm
- net MISO: track 0.00 -> 15.8 mm
- net PWM1: track 0.00 -> 14.3 mm
- net CS_: track 0.00 -> 13.9 mm
- net OUT1: track 0.00 -> 13.0 mm
- net M2-: track 0.00 -> 13.0 mm
- net M1-: track 0.00 -> 12.7 mm
- net OUT2: track 0.00 -> 12.3 mm
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- added copper zone on B.Cu, net GND
- added copper zone on F.Cu, net GND
Other:
- board outline added: 100 x 100 mm
- board text added: "NodeMcu v2 ESP8266"

Commit message: update pcb
Parts:
- removed J1: L298n_sense_connector, Connector_PinHeader_2.54mm:PinHeader_2x02_P2.54mm_Vertical
- removed J2: ACS712_connector, Connector_PinHeader_2.54mm:PinHeader_2x02_P2.54mm_Vertical
- U1: value NodeMCU1.0(ESP-12E) -> ZC563900
- moved U3 22.7 mm to (135.2, 96.2), turned to -90 degrees
- moved C8 19.6 mm to (157.5, 79.0), turned to 180 degrees
- moved C6 16.0 mm to (163.0, 79.0)
- moved C5 14.6 mm to (103.0, 79.0)
- moved C7 11.8 mm to (97.5, 79.0)
- moved R4 7.00 mm to (111.8, 121.0), turned to -90 degrees
- moved U7 1.52 mm to (100.0, 74.0)
- moved J3 1.50 mm to (88.7, 67.2)
- moved R3 1.00 mm to (109.0, 118.0)
- moved U8 0.56 mm to (160.0, 74.0)
- moved J4 0.50 mm to (171.3, 67.2)
Connections:
- U1 pad 15: +5V -> VS
- U3 pad 4: dir1_M1 -> dir2_M2
- U3 pad 5: dir1_M2 -> dir2_M1
- U3 pad 6: dir2_M1 -> dir1_M2
- U3 pad 7: dir2_M2 -> dir1_M1
- U6 pad 1: VIOUT_M1 -> VIOUT_M2
- U6 pad 2: VIOUT_M2 -> Sense_B
- U6 pad 3: unconnected-(U6-Pad3) -> Sense_A
- U6 pad 4: unconnected-(U6-Pad4) -> VIOUT_M1
Routing:
- net +3V3: track 2.00 -> 287.9 mm, vias 0 -> 5
- net VS: track 45.7 -> 208.6 mm, vias 0 -> 2
- net M1_C1: track 0.00 -> 91.9 mm
- net M1_C2: track 0.00 -> 89.0 mm
- net M2_C2: track 0.00 -> 87.2 mm
- net M2_C1: track 0.00 -> 85.1 mm
- net pwm2: track 0.00 -> 59.5 mm, vias 0 -> 1
- net VIOUT_M2: track 0.00 -> 50.2 mm
- net pwm1: track 0.00 -> 47.5 mm, vias 0 -> 1
- net VIOUT_M1: track 0.00 -> 45.8 mm
- net M1-: track 12.7 -> 49.4 mm
- net SDA: track 7.08 -> 41.7 mm
- net M2-: track 13.0 -> 44.8 mm
- net SCL: track 4.02 -> 32.7 mm
- net OUT2: track 12.3 -> 40.4 mm
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
Commit message: pcb
Parts:
- added C10: 0.1uF, Capacitor_THT:C_Disc_D4.3mm_W1.9mm_P5.00mm, F.Cu at (166.5, 115.0)
- added C11: 680uF, Capacitor_SMD:CP_Elec_8x6.9, F.Cu at (151.2, 128.2)
- added C12: 220uF, Capacitor_SMD:CP_Elec_8x6.9, F.Cu at (151.0, 146.0)
- added C9: 100uF, Capacitor_THT:CP_Radial_D6.3mm_P2.50mm, F.Cu at (162.4, 109.0)
- added D9: 1N5825, Diode_SMD:D_2010_5025Metric_Pad1.52x2.65mm_HandSolder, F.Cu at (158.0, 138.8)
- added J3: POWER, TerminalBlock_RND:TerminalBlock_RND_205-00001_1x02_P5.00mm_Horizontal, F.Cu at (163.4, 98.2)
- added J4: XT60-M, footprint:AMASS_XT60-M, F.Cu at (153.4, 93.2)
- added L1: 33uH, Inductor_SMD:L_Bourns_SRP1245A, F.Cu at (162.4, 148.8)
- added SW1: SW_DPDT_x2, Button_Switch_THT:SW_PUSH_E-Switch_FS5700DP_DPDT, F.Cu at (153.4, 109.8)
- added U9: LM2596S-5, Package_TO_SOT_SMD:TO-263-5_TabPin3, F.Cu at (162.0, 127.8)
- U4: value TXB0108DQSR -> TXB0108PWR
- moved R5 8.31 mm to (139.0, 124.0), turned to 90 degrees
- moved R6 8.31 mm to (141.0, 124.0), turned to 90 degrees
- moved R3 5.43 mm to (110.6, 112.8), turned to 90 degrees
- moved REF** 5.00 mm to (87.5, 157.5)
- moved REF** 5.00 mm to (87.5, 62.5)
- moved REF** 5.00 mm to (172.5, 157.5)
- moved REF** 5.00 mm to (172.5, 62.5)
- moved R4 4.58 mm to (110.6, 116.6)
- moved U1 4.00 mm to (130.0, 131.5)
- moved U5 4.00 mm to (130.0, 121.0)
- moved U6 3.00 mm to (130.0, 107.0)
- moved U4 0.08 mm to (124.7, 89.2)
- renumbered J3 to J1, J4 to J2
Connections:
- net pwm1 renamed pwm1_3v3
- U1 pad 26: pwm2 -> pwm2_3v3
- U3 pad 4: dir2_M2 -> dir2_M2_3v3
- U3 pad 5: dir2_M1 -> dir2_M1_3v3
- U3 pad 6: dir1_M2 -> dir1_M2_3v3
- U3 pad 7: dir1_M1 -> dir1_M1_3v3
- U4 pad 10: unconnected-(U4-Pad10) -> +3V3
- U4 pad 11: unconnected-(U4-Pad11) -> GND
- U4 pad 13: PWM2 -> unconnected-(U4-Pad13)
- U4 pad 14: DIR2_M2 -> PWM2
- U4 pad 15: GND -> DIR2_M2
- U4 pad 16: +5V -> DIR2_M1
- U4 pad 17: DIR2_M1 -> DIR1_M2
- U4 pad 18: DIR1_M2 -> DIR1_M1
- U4 pad 19: DIR1_M1 -> +5V
- U4 pad 2: dir1_M1 -> +3V3
- U4 pad 3: dir1_M2 -> dir1_M1_3v3
- U4 pad 4: dir2_M1 -> dir1_M2_3v3
- U4 pad 5: +3V3 -> dir2_M1_3v3
- U4 pad 6: +3V3 -> dir2_M2_3v3
- U4 pad 7: dir2_M2 -> pwm2_3v3
- U4 pad 8: pwm2 -> unconnected-(U4-Pad8)
Routing:
- net +5V: track 11.5 -> 250.0 mm, vias 0 -> 5
- net VS: track 208.6 -> 284.6 mm, vias 2 -> 1
- net pwm2: track 59.5 -> 0.00 mm, vias 1 -> 0
- net pwm2_3v3: track 0.00 -> 57.9 mm, vias 0 -> 1
- net Net-(J3-Pad1): track 0.00 -> 21.1 mm
- net dir1_M1_3v3: track 0.00 -> 11.7 mm
- net dir1_M1: track 11.6 -> 0.00 mm
- net Net-(D9-Pad1): track 0.00 -> 10.6 mm
- net dir1_M2: track 10.4 -> 0.00 mm
- net dir1_M2_3v3: track 0.00 -> 10.4 mm
- net dir2_M1: track 9.20 -> 0.00 mm
- net dir2_M1_3v3: track 0.00 -> 8.99 mm
- net M2_C2: track 87.2 -> 95.2 mm
- net dir2_M2_3v3: track 0.00 -> 7.63 mm
- net +3V3: track 287.9 -> 281.2 mm, vias 5 -> 2
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Other:
- board size 100 x 100 mm -> 90 x 100 mm
- board text added: "+"
- board text added: "-"
- board text added: "Turn ON/OFF"

Commit message: pcb finish
Parts:
- moved C12 13.2 mm to (150.3, 132.8)
- moved J1 12.5 mm to (100.8, 64.2), turned to 0 degrees
- moved J2 12.5 mm to (159.2, 64.2), turned to 0 degrees
- moved C7 11.8 mm to (151.9, 83.1), turned to 180 degrees
- moved C6 11.3 mm to (108.0, 83.1), turned to 0 degrees
- moved REF** 8.00 mm to (164.5, 157.5)
- moved REF** 8.00 mm to (95.5, 157.5)
- moved REF** 8.00 mm to (95.5, 62.5)
- moved REF** 8.00 mm to (164.5, 62.5)
- moved U8 7.86 mm to (157.3, 81.4), turned to 180 degrees
- moved U7 7.83 mm to (102.6, 81.4), turned to 0 degrees
- moved C11 7.36 mm to (150.3, 120.9)
- moved C4 6.65 mm to (113.3, 79.8), turned to 0 degrees
- moved L1 5.92 mm to (158.8, 144.1), turned to 180 degrees
- moved C8 5.59 mm to (151.9, 79.7)
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- renumbered C7 to C6, C6 to C7, D2 to D1, D1 to D2, D4 to D3, D3 to D4, D6 to D5, D5 to D6, D8 to D7, D7 to D8
Connections:
- U1 pad 15: VS -> +5V
Routing:
- net +3V3: track 281.2 -> 226.5 mm, vias 2 -> 4
- net +5V: track 250.0 -> 272.0 mm
- net M2-: track 43.8 -> 30.7 mm
- net M1-: track 48.3 -> 35.2 mm
- net M2_C2: track 95.2 -> 82.8 mm, vias 0 -> 2
- net VS: track 284.6 -> 295.2 mm, vias 1 -> 2
- net OUT1: track 34.0 -> 43.2 mm
- net VIOUT_M2: track 45.8 -> 37.6 mm
- net M2+: track 10.5 -> 4.10 mm
- net Net-(D9-Pad1): track 10.6 -> 16.7 mm
- net VIOUT_M1: track 44.9 -> 39.0 mm
- net M1+: track 10.4 -> 14.5 mm
- net OUT2: track 40.4 -> 44.3 mm
- net Net-(J3-Pad1): track 21.1 -> 24.3 mm
- net M1_C2: track 94.5 -> 91.4 mm
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Other:
- board size 90 x 100 mm -> 74 x 100 mm
